File: Kicad/card.kicad_pcb (KiCad board)
At the start: 2 copper layers, 21 x 51 mm, 33 parts, among them J1 USB_C_Receptacle_USB2.0_14P, J2 Conn_01x20, J3 Conn_01x20, J4 Conn_01x03, SW1 SW_Push, U1 RP2040, U2 MCP1700x-330xxTT, U3 W25Q128JVS, Y1 Crystal_GND24

Commit message: BOM
Parts:
- moved C6 1.00 mm to (159.3, 79.6)
Routing:
- net +1V1: track 6.76 -> 16.5 mm, vias 0 -> 2
- net GND: track 215.1 -> 208.2 mm, vias 12 -> 11
- net +3V3: track 97.8 -> 102.4 mm, vias 8 -> 9
- net GPIO28_ADC2: track 25.7 -> 23.1 mm
- net SWCLK: track 19.5 -> 22.2 mm
- net GPIO29_ADC3: track 28.7 -> 26.8 mm
- net GPIO9: track 6.55 -> 8.32 mm
- net GPIO14: track 20.4 -> 19.1 mm
- net GPIO8: track 9.17 -> 7.93 mm
- net GPIO13: track 14.7 -> 13.5 mm
- removed copper zone on B.Cu, net GND
- removed copper zone on F.Cu, net GND
